File: _autosave-inverteroutputboard.kicad_pcb (KiCad board)
At the start: 2 copper layers, 199.6 x 149.6 mm, 111 parts, among them P1 B+, P2 finishwinding, P3 B+, P4 startwinding, P5 CONN_02X05, Q1 Q_NMOS_GDS, Q10 Q_NMOS_GDS, Q11 Q_NMOS_GDS, Q12 Q_NMOS_GDS, Q13 Q_NMOS_GDS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

Commit message: added jumbpers
Parts:
- removed C2, C4, C5: 104/100v, Capacitors_ThroughHole:C_Disc_D7.5_P5
- removed C3, C6: 472/1kv, Capacitors_ThroughHole:C_Disc_D12_P7.75
- removed D10, D11, D12, D13, D14, D15, D16, D17, D19, D20, D21, D22, D23, D24, D7, D8, D9: 1N5819, Diodes_SMD:DO-214AB_Handsoldering
- removed D18: D_Schottky_Small, Diodes_SMD:DO-214AB_Handsoldering
- removed P2: finishwinding, Connect:1pin
- removed P3: B+, Connect:1pin
- removed P4: startwinding, Connect:1pin
- removed the P5 at (255.8, 196.4)
- removed Q10, Q11, Q12, Q13, Q14, Q15, Q16, Q17, Q18, Q19, Q20, Q21, Q22, Q23, Q24, Q7, Q8, Q9: Q_NMOS_GDS, TO_SOT_Packages_THT:TO-220_Neutral123_Horizontal_MountedFromLS_LargePads
- removed R14, R27, R40: 47R1/2w, Resistors_ThroughHole:Resistor_Horizontal_RM10mm
- removed R15, R16, R18, R19, R20, R21, R28, R29, R31, R32, R33, R34, R41, R42, R44, R45, R46, R47: 20k, Resistors_SMD:R_0603_HandSoldering
- removed R17, R22, R23, R24, R25, R26, R30, R35, R36, R37, R38, R39, R43, R48, R49, R50, R51, R52: 5.6, Resistors_SMD:R_0603_HandSoldering
- added P5: CONN_02X05, Connect:IDC_Header_Straight_10pins, F.Cu at (125.7, 83.1)
- added P5: CONN_02X05, Connect:IDC_Header_Straight_10pins, F.Cu at (38.0, 82.8)
- added REF**: Pin_Header_Straight_1x02, Pin_Headers:Pin_Header_Straight_1x02, F.Cu at (55.4, 81.0)
- D5, R10, R2: moved to F.Cu
- Q1, Q2, Q3, Q4, Q5, Q6: footprint TO_SOT_Packages_THT:TO-220_Neutral123_Horizontal_MountedFromLS_LargePads -> TO_SOT_Packages_THT:TO-220_Neutral123_Vertical
- moved D6 297.6 mm to (61.2, 70.9), turned to 90 degrees
- moved D4 294.7 mm to (72.4, 70.9), turned to 90 degrees
- moved D3 284.3 mm to (86.4, 70.4), turned to 90 degrees
- moved D2 270.5 mm to (109.2, 68.6), turned to 90 degrees
- moved D1 267.3 mm to (97.8, 69.3), turned to 90 degrees
- moved R3 263.6 mm to (70.1, 62.7), turned to 90 degrees
- moved R7 257.1 mm to (63.2, 63.4)
- moved R13 248.9 mm to (55.9, 70.9), turned to 270 degrees
- moved R8 243.0 mm to (80.8, 66.3), turned to 90 degrees
- moved R12 242.8 mm to (85.2, 61.6), turned to 270 degrees
- moved R5 242.6 mm to (92.3, 67.9), turned to 90 degrees
- moved R4 239.8 mm to (95.5, 62.0), turned to 180 degrees
- moved R11 238.2 mm to (104.5, 69.8), turned to 270 degrees
- moved P1 237.4 mm to (120.5, 51.3)
- moved R9 235.3 mm to (78.7, 71.9), turned to 270 degrees
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Connections:
- D3 pad 1: (no net) -> /PWM-C
- D3 pad 2: (no net) -> Net-(D3-Pad2)
- Q4 pad 1: Net-(Q4-Pad1) -> Net-(D3-Pad2)
- R12 pad 1: Net-(Q4-Pad1) -> Net-(D3-Pad2)
- R8 pad 1: Net-(Q4-Pad1) -> Net-(D3-Pad2)
Routing:
- net (no net): track 0.00 -> 277.9 mm
- net /endwinding: track 0.00 -> 186.1 mm, vias 0 -> 3
- net /B+: track 290.9 -> 114.5 mm
- net /PWM-C: track 0.00 -> 107.1 mm
- net Net-(D4-Pad2): track 0.00 -> 20.9 mm
- net Net-(D3-Pad2): track 0.00 -> 17.9 mm
- net Net-(D1-Pad2): track 0.00 -> 17.0 mm
- net Net-(D2-Pad2): track 0.00 -> 16.7 mm
- net Net-(D6-Pad2): track 0.00 -> 16.6 mm
- net Net-(D5-Pad2): track 0.00 -> 13.5 mm
- added copper zone on B.Cu, net /B+
- added copper zone on B.Cu, net /endwinding
Other:
- board size 199.6 x 149.6 mm -> 99.3 x 98.6 mm
- net class Default: clearance 0.2 -> 0.1
- rule trace_clearance: 0.2 -> 0.1
