File: inverteroutputboard.kicad_pcb (KiCad board)
At the start: 2 copper layers, 199.6 x 149.6 mm, 111 parts, among them P1 B+, P2 finishwinding, P3 B+, P4 startwinding, P5 CONN_02X05, Q1 Q_NMOS_GDS, Q10 Q_NMOS_GDS, Q11 Q_NMOS_GDS, Q12 Q_NMOS_GDS, Q13 Q_NMOS_GDS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

Commit message: added jumbpers
Parts:
- removed C1, C2, C4, C5: 104/100v, Capacitors_ThroughHole:C_Disc_D7.5_P5
- removed C3, C6: 472/1kv, Capacitors_ThroughHole:C_Disc_D12_P7.75
- removed D10, D11, D12, D13, D14, D15, D16, D17, D19, D20, D21, D22, D23, D24, D7, D8, D9: 1N5819, Diodes_SMD:DO-214AB_Handsoldering
- removed D18: D_Schottky_Small, Diodes_SMD:DO-214AB_Handsoldering
- removed P2: finishwinding, Connect:1pin
- removed P3: B+, Connect:1pin
- removed P4: startwinding, Connect:1pin
- removed P5: CONN_02X05, Connect:IDC_Header_Straight_10pins
- removed the Q1 at (40.6, 51.1)
- removed Q10, Q11, Q12, Q13, Q14, Q15, Q16, Q17, Q18, Q19, Q20, Q21, Q22, Q23, Q24, Q7, Q8, Q9: Q_NMOS_GDS, TO_SOT_Packages_THT:TO-220_Neutral123_Horizontal_MountedFromLS_LargePads
- removed the Q2 at (52.3, 51.1)
- removed the Q3 at (64.0, 51.1)
- removed the Q4 at (82.8, 51.1)
- removed the Q5 at (94.5, 51.1)
- removed the Q6 at (106.2, 51.1)
- removed R1, R14, R27, R40: 47R1/2w, Resistors_ThroughHole:Resistor_Horizontal_RM10mm
- removed R15, R16, R18, R19, R20, R21, R28, R29, R31, R32, R33, R34, R41, R42, R44, R45, R46, R47: 20k, Resistors_SMD:R_0603_HandSoldering
- removed R17, R22, R23, R24, R25, R26, R30, R35, R36, R37, R38, R39, R43, R48, R49, R50, R51, R52: 5.6, Resistors_SMD:R_0603_HandSoldering
- added D1: 1N5819, Diodes_SMD:DO-214AB_Handsoldering, F.Cu at (97.4, 120.7)
- added D2: 1N5819, Diodes_SMD:DO-214AB_Handsoldering, F.Cu at (108.8, 119.9)
- added D3: 1N5819, Diodes_SMD:DO-214AB_Handsoldering, F.Cu at (86.0, 121.7)
- added D4: 1N5819, Diodes_SMD:DO-214AB_Handsoldering, F.Cu at (72.0, 122.2)
- added D5: 1N5819, Diodes_SMD:DO-214AB_Handsoldering, F.Cu at (47.8, 121.7)
- added D6: 1N5819, Diodes_SMD:DO-214AB_Handsoldering, F.Cu at (60.8, 122.2)
- added P1: B+, Connect:1pin, F.Cu at (120.1, 102.6)
- added Q1: Q_NMOS_GDS, TO_SOT_Packages_THT:TO-220_Neutral123_Vertical, F.Cu at (52.2, 109.0)
- added Q1: Q_NMOS_GDS, TO_SOT_Packages_THT:TO-220_Neutral123_Vertical, F.Cu at (52.6, 57.7)
- added Q2: Q_NMOS_GDS, TO_SOT_Packages_THT:TO-220_Neutral123_Vertical, F.Cu at (64.4, 109.0)
- added Q2: Q_NMOS_GDS, TO_SOT_Packages_THT:TO-220_Neutral123_Vertical, F.Cu at (64.8, 57.7)
- added Q3: Q_NMOS_GDS, TO_SOT_Packages_THT:TO-220_Neutral123_Vertical, F.Cu at (76.6, 109.0)
- added Q3: Q_NMOS_GDS, TO_SOT_Packages_THT:TO-220_Neutral123_Vertical, F.Cu at (77.0, 57.7)
- added Q4: Q_NMOS_GDS, TO_SOT_Packages_THT:TO-220_Neutral123_Vertical, F.Cu at (88.8, 109.0)
- added Q4: Q_NMOS_GDS, TO_SOT_Packages_THT:TO-220_Neutral123_Vertical, F.Cu at (89.2, 57.7)
- added Q5: Q_NMOS_GDS, TO_SOT_Packages_THT:TO-220_Neutral123_Vertical, F.Cu at (101.0, 109.0)
- added Q5: Q_NMOS_GDS, TO_SOT_Packages_THT:TO-220_Neutral123_Vertical, F.Cu at (101.3, 57.7)
- added Q6: Q_NMOS_GDS, TO_SOT_Packages_THT:TO-220_Neutral123_Vertical, F.Cu at (113.2, 109.0)
- added Q6: Q_NMOS_GDS, TO_SOT_Packages_THT:TO-220_Neutral123_Vertical, F.Cu at (113.5, 57.7)
- added R10: 5.6, Resistors_SMD:R_0603_HandSoldering, F.Cu at (48.4, 112.8)
- added R11: 5.6, Resistors_SMD:R_0603_HandSoldering, F.Cu at (104.1, 121.2)
- added R12: 5.6, Resistors_SMD:R_0603_HandSoldering, F.Cu at (84.8, 112.9)
- added R13: 5.6, Resistors_SMD:R_0603_HandSoldering, F.Cu at (55.5, 122.2)
- added R2: 20k, Resistors_SMD:R_0603_HandSoldering, F.Cu at (53.2, 112.5)
- added R3: 20k, Resistors_SMD:R_0603_HandSoldering, F.Cu at (69.7, 114.0)
- added R4: 5.6, Resistors_SMD:R_0603_HandSoldering, F.Cu at (95.1, 113.3)
- added R5: 20k, Resistors_SMD:R_0603_HandSoldering, F.Cu at (91.9, 119.3)
- added R6: 20k, Resistors_SMD:R_0603_HandSoldering, F.Cu at (103.8, 115.6)
- added R7: 20k, Resistors_SMD:R_0603_HandSoldering, F.Cu at (62.9, 114.7)
- added R8: 20k, Resistors_SMD:R_0603_HandSoldering, F.Cu at (80.4, 117.6)
- added R9: 5.6, Resistors_SMD:R_0603_HandSoldering, F.Cu at (78.4, 123.2)
- D5, R10, R2: moved to F.Cu
- moved D6 297.6 mm to (61.2, 70.9), turned to 90 degrees
- moved D4 294.7 mm to (72.4, 70.9), turned to 90 degrees
- moved D3 284.3 mm to (86.4, 70.4), turned to 90 degrees
- moved D2 270.5 mm to (109.2, 68.6), turned to 90 degrees
- moved D1 267.3 mm to (97.8, 69.3), turned to 90 degrees
- moved R3 263.6 mm to (70.1, 62.7), turned to 90 degrees
- moved R7 257.1 mm to (63.2, 63.4)
- moved R13 248.9 mm to (55.9, 70.9), turned to 270 degrees
- moved R8 243.0 mm to (80.8, 66.3), turned to 90 degrees
- moved R12 242.8 mm to (85.2, 61.6), turned to 270 degrees
- moved R5 242.6 mm to (92.3, 67.9), turned to 90 degrees
- moved R4 239.8 mm to (95.5, 62.0), turned to 180 degrees
- moved R11 238.2 mm to (104.5, 69.8), turned to 270 degrees
- moved P1 237.4 mm to (120.5, 51.3)
- moved R9 235.3 mm to (78.7, 71.9), turned to 270 degrees
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Connections:
- D3 pad 1: (no net) -> /PWM-C
- D3 pad 2: (no net) -> Net-(D3-Pad2)
- R12 pad 1: Net-(Q4-Pad1) -> Net-(D3-Pad2)
- R8 pad 1: Net-(Q4-Pad1) -> Net-(D3-Pad2)
Routing:
- net /endwinding: track 0.00 -> 372.2 mm, vias 0 -> 6
- net /PWM-C: track 0.00 -> 214.3 mm
- net Net-(D4-Pad2): track 0.00 -> 41.7 mm
- net Net-(D3-Pad2): track 0.00 -> 35.8 mm
- net Net-(D1-Pad2): track 0.00 -> 34.1 mm
- net Net-(D2-Pad2): track 0.00 -> 33.4 mm
- net Net-(D6-Pad2): track 0.00 -> 33.2 mm
- net Net-(D5-Pad2): track 0.00 -> 26.9 mm
- net /B+: track 232.8 -> 229.0 mm
- added copper zone on B.Cu, net /B+
- added copper zone on B.Cu, net /endwinding
- removed copper zone on F.Cu, net /B+
Other:
- board size 199.6 x 149.6 mm -> 99.3 x 98.6 mm
- net class Default: clearance 0.2 -> 0.1
- rule trace_clearance: 0.2 -> 0.1

Commit message: version 0.9 caps and connectors
Parts:
- removed the D1 at (97.4, 120.7)
- removed the D2 at (108.8, 119.9)
- removed the D3 at (86.0, 121.7)
- removed the D4 at (72.0, 122.2)
- removed the D5 at (47.8, 121.7)
- removed the D6 at (60.8, 122.2)
- removed P1 (x2): B+, Connect:1pin
- removed the Q1 at (52.2, 109.0)
- removed the Q2 at (64.4, 109.0)
- removed the Q3 at (76.6, 109.0)
- removed the Q4 at (88.8, 109.0)
- removed the Q5 at (101.0, 109.0)
- removed the Q6 at (113.2, 109.0)
- removed the R10 at (48.4, 112.8)
- removed the R11 at (104.1, 121.2)
- removed the R12 at (84.8, 112.9)
- removed the R13 at (55.5, 122.2)
- removed the R2 at (53.2, 112.5)
- removed the R3 at (69.7, 114.0)
- removed the R4 at (95.1, 113.3)
- removed the R5 at (91.9, 119.3)
- removed the R6 at (103.8, 115.6)
- removed the R7 at (62.9, 114.7)
- removed the R8 at (80.4, 117.6)
- removed the R9 at (78.4, 123.2)
- added C1: 104/100v, Capacitors_ThroughHole:C_Disc_D7.5_P5, F.Cu at (128.0, 58.9)
- added C2: CP, Capacitors_ThroughHole:C_Radial_D35_L51_P10, F.Cu at (64.9, 121.5)
- added C3: CP, Capacitors_ThroughHole:C_Radial_D35_L51_P10, F.Cu at (104.4, 121.9)
- added JP1: b+, Connectors_JST:JST_EH_B02B-EH-A_02x2.50mm_Straight, F.Cu at (114.6, 85.0)
- added JP2: pwm-b, Connectors_JST:JST_EH_B02B-EH-A_02x2.50mm_Straight, F.Cu at (59.9, 84.5)
- added JP3: pwm-d, Connectors_JST:JST_EH_B02B-EH-A_02x2.50mm_Straight, F.Cu at (69.7, 84.3)
- added JP4: pwm-a, Connectors_JST:JST_EH_B02B-EH-A_02x2.50mm_Straight, F.Cu at (79.1, 84.6)
- added JP5: pwm-c, Connectors_JST:JST_EH_B02B-EH-A_02x2.50mm_Straight, F.Cu at (88.1, 84.7)
- added JP6: startwind, Connectors_JST:JST_EH_B02B-EH-A_02x2.50mm_Straight, F.Cu at (97.0, 84.7)
- added JP7: endwind, Connectors_JST:JST_EH_B02B-EH-A_02x2.50mm_Straight, F.Cu at (105.8, 85.1)
- added JP8: gnd, Connectors_JST:JST_EH_B02B-EH-A_02x2.50mm_Straight, F.Cu at (49.8, 93.2)
- added P2: CONN_02X05, Connect:IDC_Header_Straight_10pins, F.Cu at (125.1, 82.9)
- added P5: CONN_02X05, Connect:IDC_Header_Straight_10pins, F.Cu at (37.2, 82.5)
- added R1: 47R1/2w, Resistors_ThroughHole:Resistor_Horizontal_RM10mm, F.Cu at (130.8, 55.6)
- D4: value 1N5819 -> v1N5819
- Q1, Q2: value Q_NMOS_GDS -> irf4110
- moved R2 1.65 mm to (55.2, 61.2)
- turned R7 to 180 degrees
Connections:
- net /B+ renamed Net-(C1-Pad2)
- net /PWM-C renamed Net-(D1-Pad1)
- net /endwinding renamed Net-(JP6-Pad2)
Routing:
- net Net-(JP6-Pad2): track 372.2 -> 67.8 mm
- net Net-(C1-Pad2): track 229.0 -> 61.5 mm
- net GND: track 0.00 -> 109.5 mm
- net /endwinding: track 0.00 -> 106.7 mm
- net /B+: track 0.00 -> 99.3 mm
- net /startwinding: track 0.00 -> 97.3 mm
- net /PWM-D: track 0.00 -> 96.4 mm
- net /PWM-A: track 0.00 -> 93.8 mm, vias 0 -> 1
- net /PWM-B: track 0.00 -> 92.8 mm
- net /PWM-C: track 0.00 -> 91.2 mm
- net Net-(D1-Pad1): track 214.3 -> 134.9 mm
- net Net-(C2-Pad2): track 0.00 -> 39.7 mm
- net Net-(C2-Pad1): track 0.00 -> 39.7 mm
- net Net-(D4-Pad2): track 41.7 -> 20.7 mm
- net Net-(D3-Pad2): track 35.8 -> 16.6 mm
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- added copper zone on B.Cu, net Net-(C2-Pad1)
- added copper zone on F.Cu, net Net-(C2-Pad1)
- added copper zone on B.Cu, net Net-(C2-Pad2)
- added copper zone on F.Cu, net Net-(C2-Pad2)
Other:
- board text added: "Designed by Jason Devine"

Commit message: reworked plugs to make compatible with powerstar inverters and added better solder masking.
Parts:
- D4: value v1N5819 -> 1N5819
- Q1, Q2: value irf4110 -> Q_NMOS_GDS
Connections:
- P2 pad 1: GND -> /B+
- P2 pad 10: /B+ -> GND
- P2 pad 2: GND -> /B+
- P2 pad 9: /B+ -> GND
- P5 pad 1: GND -> /B+
- P5 pad 10: /B+ -> GND
- P5 pad 2: GND -> /B+
- P5 pad 9: /B+ -> GND
Routing:
- net /B+: track 99.3 -> 138.0 mm, vias 0 -> 5
- net GND: track 109.5 -> 95.5 mm
